File: Atari130MX/Atari130MX.kicad_pcb (KiCad board)
At the start: 2 copper layers, 329.2 x 129.3 mm, 84 parts, among them J0 Conn_01x26, J1 Conn_02x12_Odd_Even, J2 Conn_01x14, SW0 SW_Push_45deg, SW1 SW_Push_45deg, SW2 SW_Push_45deg, SW3 SW_Push_45deg, SW4 SW_Push_45deg, SW5 SW_Push_45deg, SW6 SW_Push_45deg, SW7 SW_Push_45deg, SW8 SW_Push_45deg, SW9 SW_Push_45deg, U1 Pico

Commit message: Modification for RetroBitLab stuff
Parts:
- removed G*** (x2): LOGO, Atari130MX:ScreamingAtTheRadio
- removed REF** (x2): AtariXE_Matrix, Atari130MX:AtariXE_Matrix
- removed REF** (x2): Decent_logo, Atari130MX:Decent_logo
- removed REF** (x2): OSH_logo, Atari130MX:OSH_logo
- removed REF0, REF01, REF02, REF03: MountingHole_3.2mm_M3, MountingHole:MountingHole_3.2mm_M3
- added JP1: SolderJumper_3_Open, Jumper:SolderJumper-3_P1.3mm_Open_RoundedPad1.0x1.5mm, F.Cu at (33.7, 77.1)
- added JP2: SolderJumper_3_Open, Jumper:SolderJumper-3_P1.3mm_Open_RoundedPad1.0x1.5mm, F.Cu at (33.6, 83.4)
- added JP3: SolderJumper_3_Open, Jumper:SolderJumper-3_P1.3mm_Open_RoundedPad1.0x1.5mm, F.Cu at (33.4, 89.8)
- added JP4: SolderJumper_3_Open, Jumper:SolderJumper-3_P1.3mm_Open_RoundedPad1.0x1.5mm, F.Cu at (33.4, 96.1)
- added L1: LOGO, RetroBit:atari_ready_8mm_rev, F.Cu at (32.8, 113.9)
- added SWSpc2: SW_Push_45deg, Atari130MX:SW_Kailh_1.50u_PCB, F.Cu at (260.7, 140.4)
- added SWSpc3: SW_Push_45deg, RetroBit:SW_Cherry_MX1A_6.25u_PCB_3d, F.Cu at (189.4, 135.3)
- J1: value Conn_02x12_Odd_Even -> Conn_01x32; footprint Atari130MX:IDC-Header_2x12_P2.54mm_Vertical -> RetroBit:MOLEX-FFC-1.25mm-RA-52044-3245
- J2: renamed from J0; footprint Connector_FFC-FPC:Molex_200528-0260_1x26-1MP_P1.00mm_Horizontal -> Atari130MX:Molex_200528-0260_1x26-1MP_P1.00mm_Horizontal
- SWSpc1: footprint Atari130MX:SW_Kailh_Atari_Space -> Atari130MX:SW_Kailh_1.25u_PCB
- U1: value Pico -> PICO_RP2040
- moved J1 77.5 mm to (342.0, 76.8)
- moved SWSpc1 71.4 mm to (115.5, 140.4)
- moved U1 9.68 mm to (54.2, 42.1)
- renumbered J2 to J3, SW7 to SW1, SW1 to SW10, SW6 to SW2, SW8 to SW3, SW5 to SW4, SW9 to SW5, SW4 to SW6, SW0 to SW7, SW3 to SW8, SW2 to SW9, SWFn3 to SWFn2, SWFn2 to SWFn3
Connections:
- net Net-(D1-Pad2) renamed LED
- net Net-(J0-Pad10) renamed COL_5
- net Net-(J0-Pad11) renamed COL_6
- net Net-(J0-Pad12) renamed ROW_3
- net Net-(J0-Pad13) renamed ROW_1
- net Net-(J0-Pad14) renamed ROW_2
- net Net-(J0-Pad15) renamed ROW_4
- net Net-(J0-Pad16) renamed COL_8
- net Net-(J0-Pad17) renamed COL_7
- net Net-(J0-Pad18) renamed ROW_6
- net Net-(J0-Pad19) renamed COL_1
- net Net-(J0-Pad21) renamed START
- net Net-(J0-Pad22) renamed SELECT
- net Net-(J0-Pad23) renamed OPTION
- net Net-(J0-Pad24) renamed RESET
- net Net-(J0-Pad4) renamed COL_2
- net Net-(J0-Pad6) renamed ROW_8
- net Net-(J0-Pad7) renamed ROW_5
- net Net-(J0-Pad8) renamed COL_3
- net Net-(J0-Pad9) renamed COL_4
- net Net-(J2-Pad10) renamed SWCLK
- net Net-(J2-Pad12) renamed GPIO26_ADC0
- net Net-(J2-Pad13) renamed GPIO27_ADC1
- net Net-(J2-Pad14) renamed GPIO28_ADC2
- net Net-(J2-Pad2) renamed 3V3_EN
- net Net-(J2-Pad3) renamed 3V3
- net Net-(J2-Pad4) renamed ADC_VREF
- net Net-(J2-Pad5) renamed AGND
- net Net-(J2-Pad6) renamed VSYS
- net Net-(J2-Pad7) renamed VBUS
- net Net-(J2-Pad8) renamed SWDIO
- net Net-(J2-Pad9) renamed RUN
- net Net-(R1-Pad1) renamed /LED-GP2
- J1 pad 1: Net-(J0-Pad1) -> POWER
- J1 pad 20: Net-(J0-Pad20) -> COL_9
- J1 pad 5: Net-(J0-Pad5) -> ROW_7
- J2 pad 1: Net-(J0-Pad1) -> POWER
- J2 pad 20: Net-(J0-Pad20) -> COL_9
- J2 pad 25: Net-(J0-Pad1) -> POWER
- J2 pad 5: Net-(J0-Pad5) -> ROW_7
- J3 pad 11: Net-(J0-Pad1) -> POWER
- SWBrk1 pad 1: Net-(J0-Pad20) -> COL_9
- SWComma1 pad 2: Net-(J0-Pad5) -> ROW_7
- SWCtl1 pad 1: Net-(J0-Pad20) -> COL_9
- SWInv1 pad 2: Net-(J0-Pad5) -> ROW_7
- SWLeftSft1 pad 1: Net-(J0-Pad20) -> Net-(JP3-Pad2)
- SWM1 pad 2: Net-(J0-Pad5) -> ROW_7
- SWN1 pad 2: Net-(J0-Pad5) -> ROW_7
- SWOption1 pad 2: GND -> Net-(JP4-Pad2)
- SWPeriod1 pad 2: Net-(J0-Pad5) -> ROW_7
- SWReset1 pad 2: GND -> Net-(JP4-Pad2)
- SWRightSft1 pad 1: Net-(J0-Pad20) -> COL_9
- SWSelect1 pad 2: GND -> Net-(JP4-Pad2)
- SWSlash1 pad 2: Net-(J0-Pad5) -> ROW_7
- SWSpc1 pad 2: Net-(J0-Pad5) -> Net-(JP1-Pad2)
- SWStart1 pad 2: GND -> Net-(JP4-Pad2)
- U1 pad 26: Net-(J0-Pad20) -> COL_9
- U1 pad 5: Net-(J0-Pad1) -> POWER
- U1 pad 7: Net-(J0-Pad5) -> ROW_7
Routing:
- net Net-(J0-Pad5): track 723.6 -> 0.00 mm
- net ROW_8: track 682.0 -> 0.00 mm, vias 1 -> 0
- net ROW_4: track 582.5 -> 0.00 mm, vias 1 -> 0
- net COL_1: track 553.2 -> 0.00 mm, vias 2 -> 0
- net COL_5: track 550.2 -> 0.00 mm, vias 1 -> 0
- net COL_4: track 546.8 -> 0.00 mm, vias 1 -> 0
- net COL_6: track 538.1 -> 0.00 mm, vias 1 -> 0
- net ROW_3: track 534.3 -> 0.00 mm, vias 1 -> 0
- net COL_7: track 531.5 -> 0.00 mm
- net ROW_5: track 521.1 -> 0.00 mm, vias 1 -> 0
- net COL_8: track 487.3 -> 0.00 mm, vias 1 -> 0
- net Net-(J0-Pad20): track 479.0 -> 0.00 mm, vias 1 -> 0
- net LED: track 464.9 -> 0.00 mm, vias 1 -> 0
- net COL_2: track 458.0 -> 0.00 mm, vias 1 -> 0
- net COL_3: track 451.2 -> 0.00 mm, vias 2 -> 0
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- removed copper zone on B.Cu, net GND
- removed copper zone on F.Cu, net GND
Other:
- board text added: "(c) Bertrand Le Roy 2021 https://github.com/bleroy/3d-junkyard/tree/main/Atari130MX https://atariage.com/forums/profile/76850-screamingattheradio/ https://www.twitch.tv/screamingattheradio https://www.youtube.com/channel/UCyaCK4oVWf1ty618W-MJcrg Modified by Gianluca Renzi 2021-12"
- board text added: "130 MX Keyboard Rev. E"
- board text added: "130MX Keyboard Rev. E"
- board text added: "ATARI / INVERT"
- board text added: "JP1 1-2 LALT JP1 2-3 ATARI SPC JP2 1-2 RALT JP2 2-3 ATARI SPC"
- board text added: "JP3 2-3 ATARI SHIFT BOTH JP3 1-2 LSHIFT JP4 1-2 ATARI GND Fn KEYS JP4 2-3 USB HID OUT_Fn"
- board text removed: "(c) Bertrand Le Roy 2021 https://github.com/bleroy/3d-junkyard/tree/main/Atari130MX https://atariage.com/forums/profile/76850-screamingattheradio/ https://www.twitch.tv/screamingattheradio https://www.youtube.com/channel/UCyaCK4oVWf1ty618W-MJcrg"
- board text removed: "130 MX Keyboard Rev. D"
- board text removed: "130MX Keyboard Rev. D"
- board text removed: "Invert"
