File: Atari130MX/Atari130MX.kicad_pcb (KiCad board)
At the start: 2 copper layers, 329.2 x 129.3 mm, 79 parts, among them J1 Conn_01x32, J2 Conn_01x26, J3 Conn_01x14, SW1 SW_Push_45deg, SW10 SW_Push_45deg, SW2 SW_Push_45deg, SW3 SW_Push_45deg, SW4 SW_Push_45deg, SW5 SW_Push_45deg, SW6 SW_Push_45deg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

Commit message: New fabrication
Parts:
- added REF**: OSHW-Logo2_9.8x8mm_SilkScreen, Symbol:OSHW-Logo2_9.8x8mm_SilkScreen, F.Cu at (279.2, 49.6)
Routing:
- net ROW_8: track 0.00 -> 614.0 mm, vias 0 -> 1
- net COL_2: track 0.00 -> 539.3 mm
- net GND: track 0.00 -> 536.0 mm
- net COL_7: track 0.00 -> 506.0 mm
- net COL_9: track 0.00 -> 468.6 mm, vias 0 -> 2
- net ROW_5: track 0.00 -> 453.2 mm, vias 0 -> 2
- net COL_8: track 0.00 -> 443.5 mm, vias 0 -> 1
- net COL_6: track 0.00 -> 439.0 mm, vias 0 -> 1
- net COL_5: track 0.00 -> 438.9 mm
- net COL_4: track 0.00 -> 438.4 mm
- net COL_1: track 0.00 -> 431.5 mm, vias 0 -> 1
- net COL_3: track 0.00 -> 428.3 mm
- net ROW_7: track 0.00 -> 418.0 mm
- net ROW_6: track 0.00 -> 416.9 mm
- net LED: track 0.00 -> 409.3 mm
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- added copper zone on B.Cu, net GND
- added copper zone on F.Cu, net GND
Other:
- board text added: "Original project by blreoy and forked to: https://github.com/gianlucarenzi/3d-junkyard/Atari130MX"
- board text added: "PLEASE DO NOT FORGET TO SET SOLDER JUMPERS!"
- board text added: "in memoriam A.S. - G.D."

Commit message: Updated with Silkscreen logos and mounting holes
Parts:
- removed REF**: OSHW-Logo2_9.8x8mm_SilkScreen, Symbol:OSHW-Logo2_9.8x8mm_SilkScreen
- added H1: MountingHole, MountingHole:MountingHole_3.2mm_M3, F.Cu at (185.8, 44.5)
- added H2: MountingHole, MountingHole:MountingHole_3.2mm_M3, F.Cu at (336.9, 40.7)
- added H3: MountingHole, MountingHole:MountingHole_3.2mm_M3, F.Cu at (336.9, 139.8)
- added H4: MountingHole, MountingHole:MountingHole_3.2mm_M3, F.Cu at (37.2, 139.8)
- added L2: LOGO, Atari130MX:AtariXE_Matrix, B.Cu at (37.2, 103.6)
- added L3: LOGO, Atari130MX:Decent_logo, F.Cu at (51.2, 141.6)
- added L4: LOGO, Atari130MX:OSH_logo, B.Cu at (30.2, 60.6)
- added L5: LOGO, Atari130MX:OSH_logo, F.Cu at (289.2, 47.6)
- added L6: LOGO, Atari130MX:ScreamingAtTheRadio, B.Cu at (168.2, 140.6)
- added L7: LOGO, Atari130MX:ScreamingAtTheRadio, F.Cu at (288.2, 139.6)
- moved L1 246.9 mm to (271.2, 49.9), turned to 0 degrees
Routing:
- net ROW_8: track 614.0 -> 0.00 mm, vias 1 -> 0
- net COL_2: track 539.3 -> 0.00 mm
- net GND: track 536.0 -> 0.00 mm
- net COL_7: track 506.0 -> 0.00 mm
- net COL_9: track 468.6 -> 0.00 mm, vias 2 -> 0
- net ROW_5: track 453.2 -> 0.00 mm, vias 2 -> 0
- net COL_8: track 443.5 -> 0.00 mm, vias 1 -> 0
- net COL_6: track 439.0 -> 0.00 mm, vias 1 -> 0
- net COL_5: track 438.9 -> 0.00 mm
- net COL_4: track 438.4 -> 0.00 mm
- net COL_1: track 431.5 -> 0.00 mm, vias 1 -> 0
- net COL_3: track 428.3 -> 0.00 mm
- net ROW_7: track 418.0 -> 0.00 mm
- net ROW_6: track 416.9 -> 0.00 mm
- net LED: track 409.3 -> 0.00 mm
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- removed copper zone on B.Cu, net GND
- removed copper zone on F.Cu, net GND
Other:
- board text added: "PLEASE DO NOT FORGET TO SET SOLDER JUMPERS BEFORE OPERATE"
- board text removed: "PLEASE DO NOT FORGET TO SET SOLDER JUMPERS!"
