File: Atari130MX/Atari130MXPlate/Atari130MXPlate.kicad_pcb (KiCad board)
At the start: 2 copper layers, 308 x 128.5 mm, 74 parts, among them SW0 SW_Push_45deg, SW1 SW_Push_45deg, SW2 SW_Push_45deg, SW3 SW_Push_45deg, SW4 SW_Push_45deg, SW5 SW_Push_45deg, SW6 SW_Push_45deg, SW7 SW_Push_45deg, SW8 SW_Push_45deg, SW9 SW_Push_45deg

Commit message: Modified for extra keys (1.25U and 1.50U) at the sides of the standard 6.25U spacebar Removed the original Atari Spacebar as it is not CherryMX compatible. Awating the STL from Axel to include it as self made printing spacebar.
The height of the PLATE + PCB must me adapted depending on which set is built.

If using original Atari Keycaps with stem adapters for Cherry MX or Kalih switches, the height of the keyboard must be
lower by 4 millimeters. Some hacks need to be done in the original Atari's case to accomplish that.

If using the original Atari Keycaps with the modified Kalih switches __AND__ the standard 6.25U + 1.25U + 1.50U switches with Cherry MX, no modifications needed.

If using the standard Cherry MX keycaps nothing has to be done to obtain the right height, but to print the function keys with Cherry MX stem.

So as you can see there is a lot of combinations to obtain the right keyboard. So everything is up to you.

I am working on a STL 3D printable case with the correct heights for spacers to fit both keycaps, so do not hold your breath if you are looking for a READY-TO-GO or DROP-IN replacement keyboard. This is not. It involves quite a hand work to obtain the final results.

Anyway it will worth the job.
Parts:
- removed SWSpc1: SW_Push_45deg, Atari130MX:SW_Hole_Atari_Space
Other:
- outline, holes or cut-outs redrawn
- board text added: "(c) Bertrand Le Roy 2021 https://github.com/bleroy/3d-junkyard/tree/main/Atari130MX https://atariage.com/forums/profile/76850-screamingattheradio/ https://www.twitch.tv/screamingattheradio https://www.youtube.com/channel/UCyaCK4oVWf1ty618W-MJcrg Modified for Cherry MX Keycaps by Gianluca Renzi RetroBit Lab"
- board text added: "130 MX Keyboard Rev. C.5"
- board text removed: "(c) Bertrand Le Roy 2021 https://github.com/bleroy/3d-junkyard/tree/main/Atari130MX https://atariage.com/forums/profile/76850-screamingattheradio/ https://www.twitch.tv/screamingattheradio https://www.youtube.com/channel/UCyaCK4oVWf1ty618W-MJcrg"
- board text removed: "130 MX Keyboard Rev. C.4"
